Commit message: clean code & update link
- change the parent link to torso

File: src/hanuman_description/urdf/hanuman.urdf.xacro (robot description, xacro)
@@ -7,6 +7,6 @@
   <!-- <xacro:include filename="$(find ${description_package})/urdf/hanuman.ros2_control.xacro" /> -->
   <xacro:include filename="$(find ${description_package})/urdf/hanuman.ros2_gazebo.xacro"/>
-  <link name="world"/>
-  <xacro:humanoid parent="world"/>
+  <xacro:robot_link link_name="torso" collision_enable="true"/>
+  <xacro:humanoid parent="torso"/>
   <!-- <xacro:humanoid_ros2_control name="humanoid_ros2_control"/> -->
 </robot>

File: src/hanuman_description/urdf/hanuman.xacro (robot description, xacro)
@@ -147,10 +147,9 @@
     <!-- full body -->
     <xacro:macro name="humanoid" params="parent">
-        <xacro:robot_link link_name="torso" collision_enable="true"/>
-        <joint name="torso_to_world" type="fixed">
+        <!-- <joint name="torso_to_world" type="fixed">
             <parent link="${parent}"/>
             <child link="torso"/>
             <origin xyz="0 0 0.9" rpy="0 0 0"/>
-        </joint>
+        </joint> -->
         <!-- <xacro:head_assem/>
         <xacro:L_arm_assem/>
