Commit message: done standing
- can control position of every joint

File: src/hanuman_description/urdf/hanuman.ros2_gazebo.xacro (robot description, xacro)
@@ -5,16 +5,4 @@
             <plugin>gazebo_ros2_control/GazeboSystem</plugin>
         </hardware>
-        <joint name="JL_hip_y">
-            <command_interface name="velocity" />
-            <command_interface name="position">
-                <param name="min" value="-3.14"/>
-                <param name="max" value="3.14"/>
-            </command_interface>
-            <state_interface name="position">
-                <param name="initial_value">0.0</param>
-            </state_interface>
-            <state_interface name="position" />
-            <state_interface name="velocity" />
-        </joint>
         <joint name="JL_hip_r">
             <command_interface name="velocity" />
@@ -65,5 +53,29 @@
             <state_interface name="velocity" />
         </joint>
+        <joint name="JL_hip_y">
+            <command_interface name="velocity" />
+            <command_interface name="position">
+                <param name="min" value="-3.14"/>
+                <param name="max" value="3.14"/>
+            </command_interface>
+            <state_interface name="position">
+                <param name="initial_value">0.0</param>
+            </state_interface>
+            <state_interface name="position" />
+            <state_interface name="velocity" />
+        </joint>
         <joint name="JL_ankle_p">
+            <command_interface name="velocity" />
+            <command_interface name="position">
+                <param name="min" value="-3.14"/>
+                <param name="max" value="3.14"/>
+            </command_interface>
+            <state_interface name="position">
+                <param name="initial_value">0.0</param>
+            </state_interface>
+            <state_interface name="position" />
+            <state_interface name="velocity" />
+        </joint>
+        <joint name="JR_hip_r">
             <command_interface name="velocity" />
             <command_interface name="position">
@@ -86,16 +98,4 @@
             </state_interface>
             <command_interface name="velocity" />
-            <state_interface name="position" />
-            <state_interface name="velocity" />
-        </joint>
-        <joint name="JR_hip_r">
-            <command_interface name="velocity" />
-            <command_interface name="position">
-                <param name="min" value="-3.14"/>
-                <param name="max" value="3.14"/>
-            </command_interface>
-            <state_interface name="position">
-                <param name="initial_value">0.0</param>
-            </state_interface>
             <state_interface name="position" />
             <state_interface name="velocity" />

Commit message: change to ignition
Encounter problems!!
- ros2 control are not available

File: src/hanuman_description/urdf/hanuman.ros2_gazebo.xacro (robot description, xacro)
@@ -3,155 +3,95 @@
     <ros2_control name="GazeboSystem" type="system">
         <hardware>
-            <plugin>gazebo_ros2_control/GazeboSystem</plugin>
+            <plugin>gz_ros2_control/GazeboSimSystem</plugin>
         </hardware>
         <joint name="JL_hip_r">
             <command_interface name="velocity" />
-            <command_interface name="position">
-                <param name="min" value="-3.14"/>
-                <param name="max" value="3.14"/>
-            </command_interface>
             <state_interface name="position">
                 <param name="initial_value">0.0</param>
             </state_interface>
-            <state_interface name="position" />
             <state_interface name="velocity" />
         </joint>
         <joint name="JL_hip_p">
             <command_interface name="velocity" />
-            <command_interface name="position">
-                <param name="min" value="-3.14"/>
-                <param name="max" value="3.14"/>
-            </command_interface>
             <state_interface name="position">
                 <param name="initial_value">0.0</param>
             </state_interface>
-            <state_interface name="position" />
             <state_interface name="velocity" />
         </joint>
         <joint name="JL_knee">
             <command_interface name="velocity" />
-            <command_interface name="position">
-                <param name="min" value="-3.14"/>
-                <param name="max" value="3.14"/>
-            </command_interface>
             <state_interface name="position">
                 <param name="initial_value">0.0</param>
             </state_interface>
-            <state_interface name="position" />
             <state_interface name="velocity" />
         </joint>
         <joint name="JL_ankle_r">
             <command_interface name="velocity" />
-            <command_interface name="position">
-                <param name="min" value="-3.14"/>
-                <param name="max" value="3.14"/>
-            </command_interface>
             <state_interface name="position">
                 <param name="initial_value">0.0</param>
             </state_interface>
-            <state_interface name="position" />
             <state_interface name="velocity" />
         </joint>
         <joint name="JL_hip_y">
             <command_interface name="velocity" />
-            <command_interface name="position">
-                <param name="min" value="-3.14"/>
-                <param name="max" value="3.14"/>
-            </command_interface>
             <state_interface name="position">
                 <param name="initial_value">0.0</param>
             </state_interface>
-            <state_interface name="position" />
             <state_interface name="velocity" />
         </joint>
         <joint name="JL_ankle_p">
             <command_interface name="velocity" />
-            <command_interface name="position">
-                <param name="min" value="-3.14"/>
-                <param name="max" value="3.14"/>
-            </command_interface>
             <state_interface name="position">
                 <param name="initial_value">0.0</param>
             </state_interface>
-            <state_interface name="position" />
             <state_interface name="velocity" />
         </joint>
         <joint name="JR_hip_r">
             <command_interface name="velocity" />
-            <command_interface name="position">
-                <param name="min" value="-3.14"/>
-                <param name="max" value="3.14"/>
-            </command_interface>
             <state_interface name="position">
                 <param name="initial_value">0.0</param>
             </state_interface>
-            <state_interface name="position" />
             <state_interface name="velocity" />
         </joint>
         <joint name="JR_hip_y">
-            <command_interface name="position">
-                <param name="min" value="-3.14"/>
-                <param name="max" value="3.14"/>
-            </command_interface>
             <state_interface name="position">
                 <param name="initial_value">0.0</param>
             </state_interface>
             <command_interface name="velocity" />
-            <state_interface name="position" />
             <state_interface name="velocity" />
         </joint>
         <joint name="JR_hip_p">
             <command_interface name="velocity" />
-            <command_interface name="position">
-                <param name="min" value="-3.14"/>
-                <param name="max" value="3.14"/>
-            </command_interface>
             <state_interface name="position">
                 <param name="initial_value">0.0</param>
             </state_interface>
-            <state_interface name="position" />
             <state_interface name="velocity" />
         </joint>
         <joint name="JR_knee">
             <command_interface name="velocity" />
-            <command_interface name="position">
-                <param name="min" value="-3.14"/>
-                <param name="max" value="3.14"/>
-            </command_interface>
             <state_interface name="position">
                 <param name="initial_value">0.0</param>
             </state_interface>
-            <state_interface name="position" />
             <state_interface name="velocity" />
         </joint>
         <joint name="JR_ankle_r">
             <command_interface name="velocity" />
-            <command_interface name="position">
-                <param name="min" value="-3.14"/>
-                <param name="max" value="3.14"/>
-            </command_interface>
             <state_interface name="position">
                 <param name="initial_value">0.0</param>
             </state_interface>
-            <state_interface name="position" />
             <state_interface name="velocity" />
         </joint>
         <joint name="JR_ankle_p">
             <command_interface name="velocity" />
-            <command_interface name="position">
-                <param name="min" value="-3.14"/>
-                <param name="max" value="3.14"/>
-            </command_interface>
             <state_interface name="position">
                 <param name="initial_value">0.0</param>
             </state_interface>
-            <state_interface name="position" />
             <state_interface name="velocity" />
         </joint>
     </ros2_control>
     <gazebo>
-        <plugin filename="libgazebo_ros2_control.so" name="gazebo_ros2_control">
+        <plugin filename="libgz_ros2_control-system.so" name="gz_ros2_control::GazeboSimROS2ControlPlugin">
             <xacro:property name="description_package" value="hanuman04" />
-            <robot_sim_type>gazebo_ros2_control/GazeboSystem</robot_sim_type>
+            <!-- <robot_sim_type>gazebo_ros2_control/GazeboSystem</robot_sim_type> -->
             <parameters>$(find ${description_package})/config/controllers.yaml</parameters>
         </plugin>

File: src/hanuman_description/urdf/hanuman.urdf.xacro (robot description, xacro)
@@ -2,11 +2,16 @@
 <robot name="hanuman" xmlns:xacro="http://ros.org/wiki/xacro">
   <!-- Include all model properties-->
-  <xacro:property name="description_package" value="hanuman04"/>
-  <xacro:include filename="$(find ${description_package})/urdf/properties.xacro"/>
+  <xacro:property name="description_package" value="hanuman04" />
+  <xacro:include filename="$(find ${description_package})/urdf/properties.xacro" />
   <xacro:include filename="$(find ${description_package})/urdf/hanuman.xacro" />
   <!-- <xacro:include filename="$(find ${description_package})/urdf/hanuman.ros2_control.xacro" /> -->
-  <xacro:include filename="$(find ${description_package})/urdf/hanuman.ros2_gazebo.xacro"/>
-  <xacro:robot_link link_name="torso" collision_enable="true"/>
-  <xacro:humanoid parent="torso"/>
+  <xacro:include filename="$(find ${description_package})/urdf/hanuman.ros2_gazebo.xacro" />
+  <!-- <link name="world"/> -->
+  <xacro:robot_link link_name="torso" collision_enable="true" />
+  <xacro:humanoid parent="torso" />
+  <!-- <joint name="base_to_torso" type="fixed">
+    <parent link="base_link"/>
+    <child link="torso"/>
+  </joint> -->
   <!-- <xacro:humanoid_ros2_control name="humanoid_ros2_control"/> -->
 </robot>

File: src/hanuman_description/urdf/hanuman.xacro (robot description, xacro)
@@ -147,8 +147,10 @@
     <!-- full body -->
     <xacro:macro name="humanoid" params="parent">
-        <!-- <joint name="torso_to_world" type="fixed">
+        <!-- <joint name="torso_to_world" type="prismatic">
             <parent link="${parent}"/>
             <child link="torso"/>
-            <origin xyz="0 0 0.9" rpy="0 0 0"/>
+            <axis xyz="0 0 1"/>
+            <limit lower="-50" upper="50" velocity="0.5" effort="1000.0"/>
+            <origin xyz="0 0 0" rpy="0 0 0"/>
         </joint> -->
         <!-- <xacro:head_assem/>

Commit message: Update Controller
usable controller added

File: src/hanuman_description/urdf/hanuman.ros2_gazebo.xacro (robot description, xacro)
@@ -5,4 +5,11 @@
             <plugin>gz_ros2_control/GazeboSimSystem</plugin>
         </hardware>
+        <joint name="JL_hip_y">
+            <command_interface name="velocity" />
+            <state_interface name="position">
+                <param name="initial_value">0.0</param>
+            </state_interface>
+            <state_interface name="velocity" />
+        </joint>
         <joint name="JL_hip_r">
             <command_interface name="velocity" />
@@ -15,5 +22,5 @@
             <command_interface name="velocity" />
             <state_interface name="position">
-                <param name="initial_value">0.0</param>
+                <param name="initial_value">1.00870663</param>
             </state_interface>
             <state_interface name="velocity" />
@@ -22,19 +29,5 @@
             <command_interface name="velocity" />
             <state_interface name="position">
-                <param name="initial_value">0.0</param>
-            </state_interface>
-            <state_interface name="velocity" />
-        </joint>
-        <joint name="JL_ankle_r">
-            <command_interface name="velocity" />
-            <state_interface name="position">
-                <param name="initial_value">0.0</param>
-            </state_interface>
-            <state_interface name="velocity" />
-        </joint>
-        <joint name="JL_hip_y">
-            <command_interface name="velocity" />
-            <state_interface name="position">
-                <param name="initial_value">0.0</param>
+                <param name="initial_value">-1.9668205</param>
             </state_interface>
             <state_interface name="velocity" />
@@ -43,9 +36,9 @@
             <command_interface name="velocity" />
             <state_interface name="position">
-                <param name="initial_value">0.0</param>
+                <param name="initial_value">0.95811387</param>
             </state_interface>
             <state_interface name="velocity" />
         </joint>
-        <joint name="JR_hip_r">
+        <joint name="JL_ankle_r">
             <command_interface name="velocity" />
             <state_interface name="position">
@@ -61,5 +54,5 @@
             <state_interface name="velocity" />
         </joint>
-        <joint name="JR_hip_p">
+        <joint name="JR_hip_r">
             <command_interface name="velocity" />
             <state_interface name="position">
@@ -68,19 +61,26 @@
             <state_interface name="velocity" />
         </joint>
+        <joint name="JR_hip_p">
+            <command_interface name="velocity" />
+            <state_interface name="position">
+                <param name="initial_value">1.00870663</param>
+            </state_interface>
+            <state_interface name="velocity" />
+        </joint>
         <joint name="JR_knee">
             <command_interface name="velocity" />
             <state_interface name="position">
-                <param name="initial_value">0.0</param>
+                <param name="initial_value">-1.9668205</param>
+            </state_interface>
+            <state_interface name="velocity" />
+        </joint>
+        <joint name="JR_ankle_p">
+            <command_interface name="velocity" />
+            <state_interface name="position">
+                <param name="initial_value">0.95811387</param>
             </state_interface>
             <state_interface name="velocity" />
         </joint>
         <joint name="JR_ankle_r">
-            <command_interface name="velocity" />
-            <state_interface name="position">
-                <param name="initial_value">0.0</param>
-            </state_interface>
-            <state_interface name="velocity" />
-        </joint>
-        <joint name="JR_ankle_p">
             <command_interface name="velocity" />
             <state_interface name="position">

Commit message: update
- real implementation
- walking trajectory problems
- joint state not working yet

File: src/hanuman_description/urdf/hanuman.ros2_gazebo.xacro (robot description, xacro)
@@ -25,5 +25,5 @@
             <state_interface name="effort"/>
             <state_interface name="position">
-                <param name="initial_value">1.00870663</param>
+                <param name="initial_value">0.0</param>
             </state_interface>
             <state_interface name="velocity" />
@@ -33,5 +33,5 @@
             <state_interface name="effort"/>
             <state_interface name="position">
-                <param name="initial_value">-1.9668205</param>
+                <param name="initial_value">0.0</param>
             </state_interface>
             <state_interface name="velocity" />
@@ -41,5 +41,5 @@
             <state_interface name="effort"/>
             <state_interface name="position">
-                <param name="initial_value">0.95811387</param>
+                <param name="initial_value">0.0</param>
             </state_interface>
             <state_interface name="velocity" />
@@ -73,5 +73,5 @@
             <state_interface name="effort"/>
             <state_interface name="position">
-                <param name="initial_value">1.00870663</param>
+                <param name="initial_value">0.0</param>
             </state_interface>
             <state_interface name="velocity" />
@@ -81,5 +81,5 @@
             <state_interface name="effort"/>
             <state_interface name="position">
-                <param name="initial_value">-1.9668205</param>
+                <param name="initial_value">0.0</param>
             </state_interface>
             <state_interface name="velocity" />
@@ -89,5 +89,5 @@
             <state_interface name="effort"/>
             <state_interface name="position">
-                <param name="initial_value">0.95811387</param>
+                <param name="initial_value">0.0</param>
             </state_interface>
             <state_interface name="velocity" />

File: src/hanuman_description/urdf/hanuman.urdf.xacro (robot description, xacro)
@@ -7,11 +7,11 @@
   <!-- <xacro:include filename="$(find ${description_package})/urdf/hanuman.ros2_control.xacro" /> -->
   <xacro:include filename="$(find ${description_package})/urdf/hanuman.ros2_gazebo.xacro" />
-  <!-- <link name="world"/> -->
+  <link name="world"/>
   <xacro:robot_link link_name="torso" collision_enable="true" />
   <xacro:humanoid parent="torso" />
-  <!-- <joint name="base_to_torso" type="fixed">
-    <parent link="base_link"/>
+  <joint name="base_to_torso" type="fixed">
+    <parent link="world"/>
     <child link="torso"/>
-  </joint> -->
+  </joint>
   <!-- <xacro:humanoid_ros2_control name="humanoid_ros2_control"/> -->
 </robot>
